File: mini-mop.kicad_pcb (KiCad board)
At the start: 2 copper layers, 100 x 50 mm, 73 parts, among them J1 Conn_Coaxial, P1 Mount, P2 Mount, Q1 BF862, Q2 BF862, U1 AD8129

Commit message: schematics elements bugs correction
Parts:
- E1, E2: value SPARK_GAP -> GAS
Changed lines of the file:
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@@
       (effects (font (size 1 1) (thickness 0.15)))
     )
-    (fp_text value SPARK_GAP (at 5.08 3.81 270) (layer F.Fab)
+    (fp_text value GAS (at 5.08 3.81 270) (layer F.Fab)
       (effects (font (size 1 1) (thickness 0.15)))
     )
@@
       (effects (font (size 1 1) (thickness 0.15)))
     )
-    (fp_text value SPARK_GAP (at 5.08 3.81 270) (layer F.Fab)
+    (fp_text value GAS (at 5.08 3.81 270) (layer F.Fab)
       (effects (font (size 1 1) (thickness 0.15)))
     )
@@
   (segment (start 97 48.5) (end 98.7 48.5) (width 0.4) (layer F.Cu) (net 3))
   (segment (start 98.7 48.5) (end 99 48.8) (width 0.4) (layer F.Cu) (net 3))
-  (segment (start 112.24 67) (end 112.24 64.24) (width 0.4) (layer B.Cu) (net 4) (status 400000))
+  (segment (start 112.24 67) (end 112.24 64.24) (width 0.4) (layer B.Cu) (net 4))
   (via (at 110 62) (size 0.6) (drill 0.4) (layers F.Cu B.Cu) (net 4))
   (segment (start 112.24 64.24) (end 110 62) (width 0.4) (layer B.Cu) (net 4))
@@
   (via (at 98.3 71.8) (size 0.6) (drill 0.4) (layers F.Cu B.Cu) (net 4))
   (segment (start 97.8 71.3) (end 98.3 71.8) (width 0.4) (layer F.Cu) (net 4))
-  (segment (start 92.75 65.2) (end 94.1 65.2) (width 0.4) (layer F.Cu) (net 4) (status 400000))
+  (segment (start 92.75 65.2) (end 94.1 65.2) (width 0.4) (layer F.Cu) (net 4))
   (via (at 108.6 70.9) (size 0.6) (drill 0.4) (layers F.Cu B.Cu) (net 4))
   (segment (start 108.6 64.6) (end 108.6 70.9) (width 0.4) (layer B.Cu) (net 4))
@@
   (segment (start 95.3 77.7) (end 99.8 77.7) (width 0.4) (layer B.Cu) (net 4))
   (via (at 99.8 77.7) (size 0.6) (drill 0.4) (layers F.Cu B.Cu) (net 4))
-  (segment (start 92.75 67.7) (end 94.5 67.7) (width 0.4) (layer F.Cu) (net 4) (status 400000))
+  (segment (start 92.75 67.7) (end 94.5 67.7) (width 0.4) (layer F.Cu) (net 4))
   (via (at 93.5 79) (size 0.6) (drill 0.4) (layers F.Cu B.Cu) (net 4))
   (segment (start 94.4 79) (end 93.5 79) (width 0.4) (layer B.Cu) (net 4))
@@
   (segment (start 94.5 67.7) (end 94.5 71.3) (width 0.4) (layer B.Cu) (net 4))
   (via (at 94.5 67.7) (size 0.6) (drill 0.4) (layers F.Cu B.Cu) (net 4))
-  (segment (start 79.8 78.45) (end 77.15 78.45) (width 0.4) (layer F.Cu) (net 4) (status 400000))
+  (segment (start 79.8 78.45) (end 77.15 78.45) (width 0.4) (layer F.Cu) (net 4))
   (via (at 77.1 81.9) (size 0.6) (drill 0.4) (layers F.Cu B.Cu) (net 4))
   (segment (start 77.1 78.5) (end 77.1 81.9) (width 0.4) (layer B.Cu) (net 4))
   (via (at 77.1 78.5) (size 0.6) (drill 0.4) (layers F.Cu B.Cu) (net 4))
   (segment (start 77.15 78.45) (end 77.1 78.5) (width 0.4) (layer F.Cu) (net 4))
-  (segment (start 79.8 78.45) (end 81.35 78.45) (width 0.4) (layer F.Cu) (net 4) (status 400000))
+  (segment (start 79.8 78.45) (end 81.35 78.45) (width 0.4) (layer F.Cu) (net 4))
   (via (at 83.5 81.8) (size 0.6) (drill 0.4) (layers F.Cu B.Cu) (net 4))
   (segment (start 83.5 78.8) (end 83.5 81.8) (width 0.4) (layer B.Cu) (net 4))
@@
   (segment (start 79.435 68.365) (end 79.4 68.4) (width 0.4) (layer F.Cu) (net 4))
   (via (at 79.4 68.4) (size 0.6) (drill 0.4) (layers F.Cu B.Cu) (net 4))
-  (segment (start 81.3 68.365) (end 79.435 68.365) (width 0.4) (layer F.Cu) (net 4) (status 400000))
+  (segment (start 81.3 68.365) (end 79.435 68.365) (width 0.4) (layer F.Cu) (net 4))
   (via (at 80.8 72.7) (size 0.6) (drill 0.4) (layers F.Cu B.Cu) (net 4))
   (segment (start 79.4 71.3) (end 80.8 72.7) (width 0.4) (layer B.Cu) (net 4))
@@
   (segment (start 82.835 68.365) (end 83.7 67.5) (width 0.4) (layer F.Cu) (net 4))
   (via (at 83.7 67.5) (size 0.6) (drill 0.4) (layers F.Cu B.Cu) (net 4))
-  (segment (start 81.3 68.365) (end 82.835 68.365) (width 0.4) (layer F.Cu) (net 4) (status 400000))
+  (segment (start 81.3 68.365) (end 82.835 68.365) (width 0.4) (layer F.Cu) (net 4))
   (via (at 86.5 64.4) (size 0.6) (drill 0.4) (layers F.Cu B.Cu) (net 4))
   (segment (start 86.4 64.5) (end 86.5 64.4) (width 0.4) (layer B.Cu) (net 4))
@@
   (via (at 91 57.6) (size 0.6) (drill 0.4) (layers F.Cu B.Cu) (net 4))
   (segment (start 91.5 57.1) (end 91 57.6) (width 0.4) (layer B.Cu) (net 4))
-  (segment (start 92.75 65.2) (end 92.75 63.65) (width 0.4) (layer F.Cu) (net 4) (status 400000))
+  (segment (start 92.75 65.2) (end 92.75 63.65) (width 0.4) (layer F.Cu) (net 4))
   (via (at 91.7 60.5) (size 0.6) (drill 0.4) (layers F.Cu B.Cu) (net 4))
   (segment (start 91.7 62.6) (end 91.7 60.5) (width 0.4) (layer F.Cu) (net 4))
